Commit message: changed urdf to correct file path for stl

File: install/learm_ros2_description/share/learm_ros2_description/urdf/learm.urdf (robot description, URDF)
Before this commit: robot learm, 12 links, 11 joints
Links:
- link base_link: geometry visual mesh filename=package://learm_ros2_description/meshes/base.stl
- link finger_left_link: geometry visual mesh filename=package://learm_ros2_description/meshes/finger.stl
- link finger_right_link: geometry visual mesh filename=package://learm_ros2_description/meshes/finger.stl
- link forearm_link: geometry visual mesh filename=package://learm_ros2_description/meshes/forearm.stl
- link grip_left_link: geometry visual mesh filename=package://learm_ros2_description/meshes/carpal-left.stl
- link grip_right_link: geometry visual mesh filename=package://learm_ros2_description/meshes/carpal-right.stl
- link hand_link: geometry visual mesh filename=package://learm_ros2_description/meshes/hand.stl
- link humerus_link: geometry visual mesh filename=package://learm_ros2_description/meshes/humerus.stl
- link shoulder_link: geometry visual mesh filename=package://learm_ros2_description/meshes/shoulder.stl
- link tendon_left_link: geometry visual mesh filename=package://learm_ros2_description/meshes/tendon.stl
- link tendon_right_link: geometry visual mesh filename=package://learm_ros2_description/meshes/tendon.stl
- link wrist_link: geometry visual mesh filename=package://learm_ros2_description/meshes/wrist.stl

File: install/learm_ros2_description/share/learm_ros2_description/urdf/learm.urdf.xacro (robot description, xacro)
@@ -1,5 +1,5 @@
 <?xml version="1.0" ?>
 <!-- =================================================================================== -->
-<!-- |    This document was autogenerated by xacro from src/learm_ros2/urdf/learm.urdf | -->
+<!-- |    This document was autogenerated by xacro from src/learm_ros2_description/urdf/learm.urdf | -->
 <!-- |    EDITING THIS FILE BY HAND IS NOT RECOMMENDED                                 | -->
 <!-- =================================================================================== -->
@@ -8,5 +8,5 @@
     <visual>
       <geometry>
-        <mesh filename="package://learm_ros2/meshes/base.stl"/>
+        <mesh filename="package://learm_ros2_description/meshes/base.stl"/>
       </geometry>
     </visual>
@@ -15,5 +15,5 @@
     <visual>
       <geometry>
-        <mesh filename="package://learm_ros2/meshes/shoulder.stl"/>
+        <mesh filename="package://learm_ros2_description/meshes/shoulder.stl"/>
       </geometry>
     </visual>
@@ -22,5 +22,5 @@
     <visual>
       <geometry>
-        <mesh filename="package://learm_ros2/meshes/humerus.stl"/>
+        <mesh filename="package://learm_ros2_description/meshes/humerus.stl"/>
       </geometry>
     </visual>
@@ -29,5 +29,5 @@
     <visual>
       <geometry>
-        <mesh filename="package://learm_ros2/meshes/forearm.stl"/>
+        <mesh filename="package://learm_ros2_description/meshes/forearm.stl"/>
       </geometry>
     </visual>
@@ -36,5 +36,5 @@
     <visual>
       <geometry>
-        <mesh filename="package://learm_ros2/meshes/wrist.stl"/>
+        <mesh filename="package://learm_ros2_description/meshes/wrist.stl"/>
       </geometry>
     </visual>
@@ -43,5 +43,5 @@
     <visual>
       <geometry>
-        <mesh filename="package://learm_ros2/meshes/hand.stl"/>
+        <mesh filename="package://learm_ros2_description/meshes/hand.stl"/>
       </geometry>
     </visual>
@@ -50,5 +50,5 @@
     <visual>
       <geometry>
-        <mesh filename="package://learm_ros2/meshes/carpal-left.stl"/>
+        <mesh filename="package://learm_ros2_description/meshes/carpal-left.stl"/>
       </geometry>
     </visual>
@@ -57,5 +57,5 @@
     <visual>
       <geometry>
-        <mesh filename="package://learm_ros2/meshes/carpal-right.stl"/>
+        <mesh filename="package://learm_ros2_description/meshes/carpal-right.stl"/>
       </geometry>
     </visual>
@@ -64,5 +64,5 @@
     <visual>
       <geometry>
-        <mesh filename="package://learm_ros2/meshes/tendon.stl"/>
+        <mesh filename="package://learm_ros2_description/meshes/tendon.stl"/>
       </geometry>
     </visual>
@@ -71,5 +71,5 @@
     <visual>
       <geometry>
-        <mesh filename="package://learm_ros2/meshes/tendon.stl"/>
+        <mesh filename="package://learm_ros2_description/meshes/tendon.stl"/>
       </geometry>
     </visual>
@@ -78,5 +78,5 @@
     <visual>
       <geometry>
-        <mesh filename="package://learm_ros2/meshes/finger.stl"/>
+        <mesh filename="package://learm_ros2_description/meshes/finger.stl"/>
       </geometry>
     </visual>
@@ -86,5 +86,5 @@
       <origin rpy="0 0 3.14159"/>
       <geometry>
-        <mesh filename="package://learm_ros2/meshes/finger.stl"/>
+        <mesh filename="package://learm_ros2_description/meshes/finger.stl"/>
       </geometry>
     </visual>
