Commit message: should've finished refactoring.. haven't tested.

File: src/learm_ros2_description/urdf/macros.xacro (robot description, xacro)
@@ -52,5 +52,5 @@
     </joint>
     <link name="grip_${side}_link">
-      <xacro:visual_collision_inertial_box size="${side == 'left' ? '2.8 0.5 5' : '-2.8 0.5 5'}" mass="1"/>
+      <xacro:visual_collision_inertial_box link_dims="${side == 'left' ? '2.8 0.5 5' : '-2.8 0.5 5'}" mass="1" link_origin="0 0 3" color="orange"/>
     </link>
   </xacro:macro>
@@ -66,5 +66,5 @@
     </joint>
     <link name="tendon_${side}_link">
-      <xacro:visual_collision_inertial_cylinder radius="0.25" length="3.8" mass="1"/>
+      <xacro:visual_collision_inertial_cylinder radius="0.25" length="3.8" mass="1" link_origin="0 0 5" color="orange"/>
     </link>
   </xacro:macro>
@@ -80,5 +80,5 @@
     </joint>
     <link name="finger_${side}_link">
-      <xacro:visual_collision_inertial_box size="${side == 'left' ? '2 0.5 6.2' : '-2 0.5 6.2'}" mass="1"/>
+      <xacro:visual_collision_inertial_box link_dims="${side == 'left' ? '2 0.5 6.2' : '-2 0.5 6.2'}" mass="1" link_origin="${side == 'left' ? '0.5 0 3' : '-0.5 0 3'}" color="red"/>
     </link>
   </xacro:macro>
@@ -118,26 +118,30 @@
   </xacro:macro>
   <!-- Macro for defining visual, collision, and inertial properties of a cylinder -->
-  <xacro:macro name="visual_collision_inertial_cylinder" params="radius length mass">
+  <xacro:macro name="visual_collision_inertial_cylinder" params="radius length mass link_origin color">
     <visual>
-      <origin xyz="0 0 0" rpy="0 0 0"/>
+      <origin xyz="${link_origin}" rpy="0 0 0"/>
       <geometry>
         <cylinder radius="${radius}" length="${length}" />
       </geometry>
-      <material name="orange"/>
+      <material name="${color}"/>
     </visual>
     <collision>
-      <origin xyz="0 0 0" rpy="0 0 0"/>
+      <origin xyz="${link_origin}" rpy="0 0 0"/>
       <geometry>
         <cylinder radius="${radius}" length="${length}" />
       </geometry>
     </collision>
-    <xacro:inertial_cylinder mass="${mass}" radius="${radius}" length="${length}"/>
+    <xacro:inertial_cylinder mass="${mass}" length="${length}" radius="${radius}">
+        <origin xyz="${link_origin}" rpy="0 0 0"/>
+    </xacro:inertial_cylinder>
   </xacro:macro>
   <!-- Macro for defining inertial properties of a cylinder -->
-  <xacro:macro name="inertial_cylinder" params="mass radius length">
+  <xacro:macro name="inertial_cylinder" params="mass length radius *origin">
     <inertial>
-      <origin xyz="0 0 0" rpy="0 0 0"/>
-      <mass value="${mass}"/>
-      <inertia ixx="${0.083333*mass*(3*radius**2+length**2)}" ixy="0" ixz="0" iyy="${0.083333*mass*(3*radius**2+length**2)}" iyz="0" izz="${0.5*mass*radius**2}"/>
+        <xacro:insert_block name="origin"/>
+        <mass value="${mass}" />
+        <inertia ixx="${(1/12) * mass * (3*radius*radius + length*length)}" ixy="0.0" ixz="0.0"
+                iyy="${(1/12) * mass * (3*radius*radius + length*length)}" iyz="0.0"
+                izz="${(1/2) * mass * (radius*radius)}" />
     </inertial>
   </xacro:macro>

File: src/learm_ros2_description/urdf/optimizedLearm.urdf.xacro (robot description, xacro)
@@ -6,13 +6,9 @@
   <xacro:base_joint_link/>
   <!-- Define the shoulder joint and link -->
-  <xacro:joint_link name="shoulder_pan" parent="base_link" child="shoulder_link" joint_origin="0 7 7" axis="0 0 1" lower="${-pi/2}" upper="${pi/2}" velocity="100" effort="100" link_dims="4.2 4.1 2.2" mass="50"/>
-  <!-- Define the humerus joint and link -->
-  <xacro:joint_link name="elbow" parent="shoulder_link" child="humerus_link" joint_origin="0 1.5 7" axis="1 0 0" lower="${-pi/2}" upper="${pi/2}" velocity="100" effort="100" link_dims="5.5 3 13" mass="200"/>
-  <!-- Define the forearm joint and link -->
-  <xacro:joint_link name="wrist_flex" parent="humerus_link" child="forearm_link" joint_origin="0 1.5 13" axis="1 0 0" lower="${-pi/2}" upper="${pi/2}" velocity="100" effort="100" link_dims="5.5 3 11" mass="200"/>
-  <!-- Define the wrist joint and link -->
-  <xacro:joint_link name="wrist_roll" parent="forearm_link" child="wrist_link" joint_origin="0 0 11" axis="0 0 1" lower="${-pi/2}" upper="${pi/2}" velocity="100" effort="100" link_dims="5.5 5 7.5" mass="200"/>
-  <!-- Define the hand joint and link -->
-  <xacro:joint_link name="wrist_flex" parent="wrist_link" child="hand_link" joint_origin="0 0 7.5" axis="0 0 1" lower="${-pi/2}" upper="${pi/2}" velocity="100" effort="100" link_dims="5.5 5 4" mass="200"/>
+  <xacro:joint_link name="shoulder_pan" parent="base_link" child="shoulder_link" joint_origin="0 7 7" axis="0 0 1" lower="${-pi/2}" upper="${pi/2}" velocity="100" effort="100" link_dims="4.2 4.1 2.2" mass="50" link_origin="0 0 0" color="black"/>
+  <xacro:joint_link name="shoulder_lift" parent="shoulder_link" child="humerus_link" joint_origin="0 1.05 1.1" axis="-1 0 0" lower="${-pi/2}" upper="${pi/2}" velocity="100" effort="100" link_dims="5.5 3 13" mass="200" link_origin="0 1.5 7" color="blue"/>
+  <xacro:joint_link name="elbow" parent="humerus_link" child="forearm_link" joint_origin="0 1.5 13" axis="1 0 0" lower="${-pi/2}" upper="${pi/2}" velocity="100" effort="100" link_dims="5.5 3 11" mass="200" link_origin="0 0 5.5" color="blue"/>
+  <xacro:joint_link name="wrist_flex" parent="forearm_link" child="wrist_link" joint_origin="0 0 11" axis="1 0 0" lower="${-pi/2}" upper="${pi/2}" velocity="100" effort="100" link_dims="5.5 5 7.5" mass="200" link_origin="0 1.5 3.25" color="blue"/>
+  <xacro:joint_link name="wrist_roll" parent="wrist_link" child="hand_link" joint_origin="0 0 7.5" axis="0 0 1" lower="${-pi/2}" upper="${pi/2}" velocity="100" effort="100" link_dims="5.5 5 4" mass="200" link_origin="0 -1.5 2" color="blue"/>
   <!-- Define the grip joints and links -->
   <xacro:grip_joint_link side="left"/>

Commit message: refactoring doesn't work. Something weird with parameters it doesn't like. Next time just adjust the claw to face the other direction.

File: src/learm_ros2_description/urdf/macros.xacro (robot description, xacro)
@@ -98,11 +98,5 @@
       </geometry>
     </collision>
-    <!-- Split the link_dims string into a list of numbers -->
-    <xacro:property name="dims_list" value="xacro:split(string(${link_dims}), ' ')" />
-    <!-- Extract individual components (x, y, z) -->
-    <xacro:property name="x" value="${dims_list[0]}" />
-    <xacro:property name="y" value="${dims_list[1]}" />
-    <xacro:property name="z" value="${dims_list[2]}" />
-    <xacro:inertial_box mass="${mass}" x="${x}" y="${y}" z="${z}">
+    <xacro:inertial_box mass="${mass}" x="${link_dims[0]}" y="${link_dims[1]}" z="${link_dims[2]}">
         <origin xyz="link_origin" rpy="0 0 0"/>
     </xacro:inertial_box>
