Commit message: fixed bounds of spinning joints.

File: src/learm_ros2_description/urdf/newLearm.urdf.xacro (robot description, xacro)
@@ -42,6 +42,5 @@
         <child link="shoulder_link"/>
         <axis xyz="0 0 1"/>
-        <limit effort="100" lower="-3.14159" upper="3.14159" velocity="1.0"/>
-        <limit effort="100" lower="-6.28318" upper="6.28318" velocity="1.0"/>
+        <limit lower="${-pi/2}" upper="${pi/2}" velocity="100" effort="100"/>
     </joint>
     <!-- small plate for the servo which is art 2 -->
@@ -159,6 +158,5 @@
         <child link="hand_link"/>
         <axis xyz="0 0 1"/>
-        <limit effort="100" lower="-3.14159" upper="3.14159" velocity="1.0"/>
-        <limit effort="100" lower="-6.28318" upper="6.28318" velocity="1.0"/>
+        <limit effort="100" lower="${-pi/2}" upper="${-pi/2}" velocity="1.0"/>
     </joint>
     <link name="hand_link">

Commit message: The orientation of the wrist model needs to be changed. The rotation needs to be 90degrees... go back to what it was when you first started :///

File: src/learm_ros2_description/urdf/newLearm.urdf.xacro (robot description, xacro)
@@ -70,5 +70,5 @@
         <parent link="shoulder_link"/>
         <child link="humerus_link"/>
-        <axis xyz="1 0 0"/>
+        <axis xyz="-1 0 0"/>
         <limit lower="${-pi/2}" upper="${pi/2}" velocity="100" effort="100"/>
     </joint>
@@ -158,5 +158,5 @@
         <child link="hand_link"/>
         <axis xyz="0 0 1"/>
-        <limit effort="100" lower="${-pi/2}" upper="${-pi/2}" velocity="1.0"/>
+        <limit effort="100" lower="${-pi/2}" upper="${pi/2}" velocity="1.0"/>
     </joint>
     <link name="hand_link">

Commit message: incremental changes to the urdf to modularize it and make it more readable. Not done and need to adjust orientation of hand still

File: src/learm_ros2_description/urdf/newLearm.urdf.xacro (robot description, xacro)
@@ -1,13 +1,8 @@
 <?xml version="1.0"?>
 <robot xmlns:xacro="http://www.ros.org/wiki/xacro"  name="robot">
-    <!-- This is an example of a URDF. -->
-    <!-- As we move through the file, new things to note will be pointed out. -->
-    <!-- It's not meant an example of GOOD design, but an example of some of the various features of URDF/xacro. -->
-    <!-- This will include all the contents of example_include.xacro first. Go check it out! -->
+    <!-- This will include all the contents of example_include.xacro first. -->
     <xacro:include filename="example_include.xacro" />
     <!-- This first link called "world" is empty -->
     <link name="world"></link>
-    <!-- A simple fixed joint from our empty world link, to our base. -->
-    <!-- The base origin is offset from the world origin. -->
     <joint name="base_joint" type="fixed">
         <origin xyz="1.5 1.0 0" rpy="0 0 0"/>
@@ -15,5 +10,4 @@
         <child link="base_link"/>
     </joint>
-    <!-- base, z offset to sit the object on the ground -->
     <link name="base_link">
         <visual>
@@ -36,5 +30,4 @@
         </xacro:inertial_box>
     </link>
-    <!-- - articulation one joint -->
     <joint name="shoulder_pan" type="revolute">
         <origin xyz="0 7 7" rpy="0 0 0"/>
@@ -44,5 +37,4 @@
         <limit lower="${-pi/2}" upper="${pi/2}" velocity="100" effort="100"/>
     </joint>
-    <!-- small plate for the servo which is art 2 -->
     <link name="shoulder_link">
         <visual>
@@ -65,5 +57,4 @@
         </xacro:inertial_box>
     </link>
-    <!-- articulation two joint -->
     <joint name="shoulder_lift" type="revolute">
         <origin xyz="0 1.05 1.1" rpy="0 0 0"/>
@@ -73,7 +64,4 @@
         <limit lower="${-pi/2}" upper="${pi/2}" velocity="100" effort="100"/>
     </joint>
-    <!-- slider_link is the box skimming across the top of the base. Its parameters are similar to the base_link, however: -->
-    <!-- - Instead of explicitly describing a colour, it uses the named material "blue". It knows about "blue" that material was included in example_include.xacro. -->
-    <!-- - Instead of explicitly describing the inertia, we use a macro that was defined in the example_include.xacro -->
     <link name="humerus_link">
         <visual>
@@ -94,7 +82,4 @@
         </xacro:inertial_box>
     </link>
-    <!-- arm_joint describes the rotation of the arm and is centred around the top corner of the slider box. -->
-    <!-- - The axis of rotation is -1 in Y, so that positive is "up" -->
-    <!-- - The upper limit uses xacro's mathematical features -->
     <joint name="elbow" type="revolute">
         <origin xyz="0 1.5 13" rpy="0 0 0"/>
@@ -104,10 +89,4 @@
         <limit lower="${-pi/2}" upper="${pi/2}" velocity="100" effort="100"/>
     </joint>
-    <!-- arm_link describes the arm -->
-    <!-- - We use the "property" feature to define the arm length and radius and use them multiple times -->
-    <!-- - The visual/collision origin is set to halfway along the length (similar to the box), but also with a rotation (again using the mathematical features). -->
-    <!--   This is because the cylinder extends along the Z axis by default, but we want it to be along the X axis (when the joint is at 0) -->
-    <xacro:property name="arm_length" value="11" />
-    <xacro:property name="arm_radius" value="2.75" />
     <link name="forearm_link">
         <visual>

Commit message: Robot urdf fixed. Next step: Moveit setup assistant.

File: src/learm_ros2_description/urdf/newLearm.urdf.xacro (robot description, xacro)
@@ -141,18 +141,18 @@
     <link name="hand_link">
         <visual>
-            <origin xyz="0 -1.5 2" rpy="0 0 0"/>
-            <geometry>
-                <box size="5.5 5 4" />
+            <origin xyz="1.5 -1.5 2" rpy="0 0 0"/>
+            <geometry>
+                <box size="5 5.5 4" />
             </geometry>
             <material name="blue" />
         </visual>
         <collision>
-            <origin xyz="0 -1.5 2" rpy="0 0 0"/>
-            <geometry>
-                <box size="5.5 5 4" />
-            </geometry>
-        </collision>
-        <xacro:inertial_box mass="200" x="5.5" y="5" z="4">
-            <origin xyz="0 -1.5 2" rpy="0 0 0"/>
+            <origin xyz="1.5 -1.5 2" rpy="0 0 0"/>
+            <geometry>
+                <box size="5 5.5 4" />
+            </geometry>
+        </collision>
+        <xacro:inertial_box mass="200" x="5" y="5.5" z="4">
+            <origin xyz="1.5 -1.5 2" rpy="0 0 0"/>
         </xacro:inertial_box>
     </link>
@@ -161,6 +161,6 @@
         <parent link="hand_link"/>
         <child link="grip_left_link"/>
-        <origin xyz="-1.5 0 3" rpy="0 -1.57 0"/>
-        <axis xyz="0 -1 0"/>
+        <origin xyz="0 0 3" rpy="-1.57 0 0"/>
+        <axis xyz="-1 0 0"/>
         <limit lower="-1.57" upper="0" effort="1000" velocity="0.5"/>
     </joint>
@@ -168,6 +168,6 @@
         <parent link="hand_link"/>
         <child link="grip_right_link"/>
-        <origin xyz="1.5 0 3" rpy="0 1.57 0"/>
-        <axis xyz="0 -1 0"/>
+        <origin xyz="0 -3 3" rpy="1.57 0 0"/>
+        <axis xyz="-1 0 0"/>
         <limit lower="0" upper="1.57" effort="1000" velocity="0.5"/>
         <mimic joint="grip_left" multiplier="-1"/>
@@ -177,5 +177,5 @@
             <origin xyz="0 0 3" rpy="0 0 0"/>
             <geometry>
-                <box size="2.8 0.5 5" />
+                <box size="0.5 -2.8 5" />
             </geometry>
             <material name="orange" />
@@ -184,8 +184,8 @@
             <origin xyz="0 0 3" rpy="0 0 0"/>
             <geometry>
-                <box size="2.8 0.5 5" />
-            </geometry>
-        </collision>
-        <xacro:inertial_box mass="1" x="2.8" y="0.5" z="5">
+                <box size="0.5 -2.8 5" />
+            </geometry>
+        </collision>
+        <xacro:inertial_box mass="1" x="0.5" y="-2.8" z="5">
             <origin xyz="0 0 3" rpy="0 0 0"/>
         </xacro:inertial_box>
@@ -195,5 +195,5 @@
             <origin xyz="0 0 3" rpy="0 0 0"/>
             <geometry>
-                <box size="-2.8 0.5 5" />
+                <box size="0.5 2.8 5" />
             </geometry>
             <material name="orange" />
@@ -202,8 +202,8 @@
             <origin xyz="0 0 3" rpy="0 0 0"/>
             <geometry>
-                <box size="-2.8 0.5 5" />
-            </geometry>
-        </collision>
-        <xacro:inertial_box mass="1" x="-2.8" y="0.5" z="5">
+                <box size="0.5 2.8 5" />
+            </geometry>
+        </collision>
+        <xacro:inertial_box mass="1" x="0.5" y="2.8" z="5">
             <origin xyz="0 0 3" rpy="0 0 0"/>
         </xacro:inertial_box>
@@ -213,6 +213,6 @@
         <parent link="hand_link"/>
         <child link="tendon_left_link"/>
-        <origin xyz="-0.5 0 5" rpy="0 -1.57 0"/>
-        <axis xyz="0 -1 0"/>
+        <origin xyz="0 -2 5" rpy="1.57 0 0"/>
+        <axis xyz="1 0 0"/>
         <limit lower="-1.57" upper="0" effort="1000" velocity="0.5"/>
         <mimic joint="grip_left"/>
@@ -221,6 +221,6 @@
         <parent link="hand_link"/>
         <child link="tendon_right_link"/>
-        <origin xyz="0.5 0 5" rpy="0 1.57 0"/>
-        <axis xyz="0 -1 0"/>
+        <origin xyz="0 -1 5" rpy="-1.57 0 0"/>
+        <axis xyz="1 0 0"/>
         <limit lower="0" upper="1.57" effort="1000" velocity="0.5"/>
         <mimic joint="grip_left" multiplier="-1"/>
@@ -266,6 +266,6 @@
         <parent link="grip_left_link"/>
         <child link="finger_left_link"/>
-        <origin xyz="0 0 5.5" rpy="0 1.57 0"/>
-        <axis xyz="0 -1 0"/>
+        <origin xyz="0 0 5.5" rpy="1.57 0 0"/>
+        <axis xyz="-1 0 0"/>
         <limit lower="-1.57" upper="0" effort="1000" velocity="0.5"/>
         <mimic joint="grip_left" multiplier="-1"/>
@@ -274,6 +274,6 @@
         <parent link="grip_right_link"/>
         <child link="finger_right_link"/>
-        <origin xyz="0 0 5.5" rpy="0 -1.57 0"/>
-        <axis xyz="0 -1 0"/>
+        <origin xyz="0 0 5.5" rpy="-1.57 0 0"/>
+        <axis xyz="-1 0 0"/>
         <limit lower="0" upper="1.57" effort="1000" velocity="0.5"/>
         <mimic joint="grip_left"/>
@@ -281,36 +281,36 @@
     <link name="finger_left_link">
         <visual>
-            <origin xyz="0.5 0 3" rpy="0 0 0"/>
-            <geometry>
-                <box size="2 0.5 6.2" />
+            <origin xyz="0 -0.5 3" rpy="0 0 0"/>
+            <geometry>
+                <box size="0.5 2 6.2" />
             </geometry>
             <material name="red" />
         </visual>
         <collision>
-            <origin xyz="0.5 0 3" rpy="0 0 0"/>
-            <geometry>
-                <box size="2 0.5 6.2" />
-            </geometry>
-        </collision>
-        <xacro:inertial_box mass="1" x="2" y="0.5" z="6.2">
-            <origin xyz="0.5 0 3" rpy="0 0 0"/>
+            <origin xyz="0 -0.5 3" rpy="0 0 0"/>
+            <geometry>
+                <box size="0.5 2 6.2" />
+            </geometry>
+        </collision>
+        <xacro:inertial_box mass="1" x="0.5" y="2" z="6.2">
+            <origin xyz="0 -0.5 3" rpy="0 0 0"/>
         </xacro:inertial_box>
     </link>
     <link name="finger_right_link">
         <visual>
-            <origin xyz="-0.5 0 3" rpy="0 0 0"/>
-            <geometry>
-                <box size="-2 0.5 6.2" />
+            <origin xyz="0 0.5 3" rpy="0 0 0"/>
+            <geometry>
+                <box size="0.5 -2 6.2" />
             </geometry>
             <material name="red" />
         </visual>
         <collision>
-            <origin xyz="-0.5 0 3" rpy="0 0 0"/>
-            <geometry>
-                <box size="-2 0.5 6.2" />
-            </geometry>
-        </collision>
-        <xacro:inertial_box mass="1" x="-2" y="0.5" z="6.2">
-            <origin xyz="-0.5 0 3" rpy="0 0 0"/>
+            <origin xyz="0 0.5 3" rpy="0 0 0"/>
+            <geometry>
+                <box size="0.5 -2 6.2" />
+            </geometry>
+        </collision>
+        <xacro:inertial_box mass="1" x="0.5" y="-2" z="6.2">
+            <origin xyz="0 0.5 3" rpy="0 0 0"/>
         </xacro:inertial_box>
     </link>
