Commit message: Added correctly scaled urdf!

File: src/learm_ros2_description/urdf/scaledLearm.urdf.xacro (robot description, xacro)
@@ -6,5 +6,5 @@
     <link name="world"></link>
     <joint name="base_joint" type="fixed">
-        <origin xyz="1.5 1.0 0" rpy="0 0 0"/>
+        <origin xyz="0.015 0.010 0" rpy="0 0 0"/>
         <parent link="world"/>
         <child link="base_link"/>
@@ -12,7 +12,7 @@
     <link name="base_link">
         <visual>
-            <origin xyz="0 0 3.5" rpy="0 0 0"/>
-            <geometry>
-                <box size="16 29 7" />
+            <origin xyz="0 0 0.035" rpy="0 0 0"/>
+            <geometry>
+                <box size="0.16 0.29 0.07" />
             </geometry>
             <material name="green">
@@ -21,15 +21,15 @@
         </visual>
         <collision>
-            <origin xyz="0 0 3.5" rpy="0 0 0"/>
-            <geometry>
-                <box size="16 29 7" />
-            </geometry>
-        </collision>
-        <xacro:inertial_box mass="500" x="16" y="29" z="7">
-            <origin xyz="0 0 3.5" rpy="0 0 0"/>
+            <origin xyz="0 0 0.035" rpy="0 0 0"/>
+            <geometry>
+                <box size="0.16 0.29 0.07" />
+            </geometry>
+        </collision>
+        <xacro:inertial_box mass="500" x="0.16" y="0.29" z="0.07">
+            <origin xyz="0 0 0.035" rpy="0 0 0"/>
         </xacro:inertial_box>
     </link>
     <joint name="shoulder_pan" type="revolute">
-        <origin xyz="0 7 7" rpy="0 0 0"/>
+        <origin xyz="0 0.07 0.07" rpy="0 0 0"/>
         <parent link="base_link"/>
         <child link="shoulder_link"/>
@@ -41,5 +41,5 @@
             <origin xyz="0 0 0" rpy="0 0 0"/>
             <geometry>
-                <box size="4.2 4.1 2.2" />
+                <box size="0.042 0.041 0.022" />
             </geometry>
             <material name="black">
@@ -50,13 +50,13 @@
             <origin xyz="0 0 0" rpy="0 0 0"/>
             <geometry>
-                <box size="4.2 4.1 2.2" />
-            </geometry>
-        </collision>
-        <xacro:inertial_box mass="50" x="4.2" y="4.1" z="2.2">
+                <box size="0.042 0.041 0.022" />
+            </geometry>
+        </collision>
+        <xacro:inertial_box mass="50" x="0.042" y="0.041" z="0.022">
             <origin xyz="0 0 0" rpy="0 0 0"/>
         </xacro:inertial_box>
     </link>
     <joint name="shoulder_lift" type="revolute">
-        <origin xyz="0 1.05 1.1" rpy="0 0 0"/>
+        <origin xyz="0 0.0105 0.011" rpy="0 0 0"/>
         <parent link="shoulder_link"/>
         <child link="humerus_link"/>
@@ -66,22 +66,22 @@
     <link name="humerus_link">
         <visual>
-            <origin xyz="0 1.5 7" rpy="0 0 0"/>
-            <geometry>
-                <box size="5.5 3 13" />
+            <origin xyz="0 0.015 0.07" rpy="0 0 0"/>
+            <geometry>
+                <box size="0.055 0.03 0.13" />
             </geometry>
             <material name="blue" />
         </visual>
         <collision>
-            <origin xyz="0 1.5 7" rpy="0 0 0"/>
-            <geometry>
-                <box size="5.5 3 13" />
-            </geometry>
-        </collision>
-        <xacro:inertial_box mass="200" x="5.5" y="3" z="13">
-            <origin xyz="0 1.5 7" rpy="0 0 0"/>
+            <origin xyz="0 0.015 0.07" rpy="0 0 0"/>
+            <geometry>
+                <box size="0.055 0.03 0.13" />
+            </geometry>
+        </collision>
+        <xacro:inertial_box mass="200" x="0.055" y="0.03" z="0.13">
+            <origin xyz="0 0.015 0.07" rpy="0 0 0"/>
         </xacro:inertial_box>
     </link>
     <joint name="elbow" type="revolute">
-        <origin xyz="0 1.5 13" rpy="0 0 0"/>
+        <origin xyz="0 0.015 0.13" rpy="0 0 0"/>
         <parent link="humerus_link"/>
         <child link="forearm_link"/>
@@ -91,22 +91,22 @@
     <link name="forearm_link">
         <visual>
-            <origin xyz="0 0 5.5" rpy="0 0 0"/>
-            <geometry>
-                <box size="5.5 3 11" />
+            <origin xyz="0 0 0.055" rpy="0 0 0"/>
+            <geometry>
+                <box size="0.055 0.03 0.11" />
             </geometry>
             <material name="blue" />
         </visual>
         <collision>
-            <origin xyz="0 0 5.5" rpy="0 0 0"/>
-            <geometry>
-                <box size="5.5 3 11" />
-            </geometry>
-        </collision>
-        <xacro:inertial_box mass="200" x="5.5" y="3" z="11">
-            <origin xyz="0 0 5.5" rpy="0 0 0"/>
+            <origin xyz="0 0 0.055" rpy="0 0 0"/>
+            <geometry>
+                <box size="0.055 0.03 0.11" />
+            </geometry>
+        </collision>
+        <xacro:inertial_box mass="200" x="0.055" y="0.03" z="0.11">
+            <origin xyz="0 0 0.055" rpy="0 0 0"/>
         </xacro:inertial_box>
     </link>
     <joint name="wrist_flex" type="revolute">
-        <origin xyz="0 0 11" rpy="0 0 0"/>
+        <origin xyz="0 0 0.11" rpy="0 0 0"/>
         <parent link="forearm_link"/>
         <child link="wrist_link"/>
@@ -116,22 +116,22 @@
     <link name="wrist_link">
         <visual>
-            <origin xyz="0 1.5 3.25" rpy="0 0 0"/>
-            <geometry>
-                <box size="5.5 5 7.5" />
+            <origin xyz="0 0.015 0.0325" rpy="0 0 0"/>
+            <geometry>
+                <box size="0.055 0.05 0.075" />
             </geometry>
             <material name="blue" />
         </visual>
         <collision>
-            <origin xyz="0 1.5 3.25" rpy="0 0 0"/>
-            <geometry>
-                <box size="5.5 5 7.5" />
-            </geometry>
-        </collision>
-        <xacro:inertial_box mass="200" x="5.5" y="5" z="7.5">
-            <origin xyz="0 1.5 3.25" rpy="0 0 0"/>
+            <origin xyz="0 0.015 0.0325" rpy="0 0 0"/>
+            <geometry>
+                <box size="0.055 0.05 0.075" />
+            </geometry>
+        </collision>
+        <xacro:inertial_box mass="200" x="0.055" y="0.05" z="0.075">
+            <origin xyz="0 0.015 0.0325" rpy="0 0 0"/>
         </xacro:inertial_box>
     </link>
     <joint name="wrist_roll" type="revolute">
-        <origin xyz="0 0 7.5" rpy="0 0 0"/>
+        <origin xyz="0 0 0.075" rpy="0 0 0"/>
         <parent link="wrist_link"/>
         <child link="hand_link"/>
@@ -141,18 +141,18 @@
     <link name="hand_link">
         <visual>
-            <origin xyz="1.5 -1.5 2" rpy="0 0 0"/>
-            <geometry>
-                <box size="5 5.5 4" />
+            <origin xyz="0.015 -0.015 0.02" rpy="0 0 0"/>
+            <geometry>
+                <box size="0.05 0.055 0.04" />
             </geometry>
             <material name="blue" />
         </visual>
         <collision>
-            <origin xyz="1.5 -1.5 2" rpy="0 0 0"/>
-            <geometry>
-                <box size="5 5.5 4" />
-            </geometry>
-        </collision>
-        <xacro:inertial_box mass="200" x="5" y="5.5" z="4">
-            <origin xyz="1.5 -1.5 2" rpy="0 0 0"/>
+            <origin xyz="0.015 -0.015 0.02" rpy="0 0 0"/>
+            <geometry>
+                <box size="0.05 0.055 0.04" />
+            </geometry>
+        </collision>
+        <xacro:inertial_box mass="200" x="0.05" y="0.055" z="0.04">
+            <origin xyz="0.015 -0.015 0.02" rpy="0 0 0"/>
         </xacro:inertial_box>
     </link>
@@ -161,5 +161,5 @@
         <parent link="hand_link"/>
         <child link="grip_left_link"/>
-        <origin xyz="0 0 3" rpy="-1.57 0 0"/>
+        <origin xyz="0 0 0.03" rpy="-1.57 0 0"/>
         <axis xyz="-1 0 0"/>
         <limit lower="-1.57" upper="0" effort="1000" velocity="0.5"/>
@@ -168,5 +168,5 @@
         <parent link="hand_link"/>
         <child link="grip_right_link"/>
-        <origin xyz="0 -3 3" rpy="1.57 0 0"/>
+        <origin xyz="0 -0.03 0.03" rpy="1.57 0 0"/>
         <axis xyz="-1 0 0"/>
         <limit lower="0" upper="1.57" effort="1000" velocity="0.5"/>
@@ -175,36 +175,36 @@
     <link name="grip_left_link">
         <visual>
-            <origin xyz="0 0 3" rpy="0 0 0"/>
-            <geometry>
-                <box size="0.5 -2.8 5" />
+            <origin xyz="0 0 0.03" rpy="0 0 0"/>
+            <geometry>
+                <box size="0.005 -0.028 0.05" />
             </geometry>
             <material name="orange" />
         </visual>
         <collision>
-            <origin xyz="0 0 3" rpy="0 0 0"/>
-            <geometry>
-                <box size="0.5 -2.8 5" />
-            </geometry>
-        </collision>
-        <xacro:inertial_box mass="1" x="0.5" y="-2.8" z="5">
-            <origin xyz="0 0 3" rpy="0 0 0"/>
+            <origin xyz="0 0 0.03" rpy="0 0 0"/>
+            <geometry>
+                <box size="0.005 -0.028 0.05" />
+            </geometry>
+        </collision>
+        <xacro:inertial_box mass="1" x="0.005" y="-0.028" z="0.05">
+            <origin xyz="0 0 0.03" rpy="0 0 0"/>
         </xacro:inertial_box>
     </link>
     <link name="grip_right_link">
         <visual>
-            <origin xyz="0 0 3" rpy="0 0 0"/>
-            <geometry>
-                <box size="0.5 2.8 5" />
+            <origin xyz="0 0 0.03" rpy="0 0 0"/>
+            <geometry>
+                <box size="0.005 0.028 0.05" />
             </geometry>
             <material name="orange" />
         </visual>
         <collision>
-            <origin xyz="0 0 3" rpy="0 0 0"/>
-            <geometry>
-                <box size="0.5 2.8 5" />
-            </geometry>
-        </collision>
-        <xacro:inertial_box mass="1" x="0.5" y="2.8" z="5">
-            <origin xyz="0 0 3" rpy="0 0 0"/>
+            <origin xyz="0 0 0.03" rpy="0 0 0"/>
+            <geometry>
+                <box size="0.005 0.028 0.05" />
+            </geometry>
+        </collision>
+        <xacro:inertial_box mass="1" x="0.005" y="0.028" z="0.05">
+            <origin xyz="0 0 0.03" rpy="0 0 0"/>
         </xacro:inertial_box>
     </link>
@@ -213,5 +213,5 @@
         <parent link="hand_link"/>
         <child link="tendon_left_link"/>
-        <origin xyz="0 -2 5" rpy="1.57 0 0"/>
+        <origin xyz="0 -0.02 0.05" rpy="1.57 0 0"/>
         <axis xyz="1 0 0"/>
         <limit lower="-1.57" upper="0" effort="1000" velocity="0.5"/>
@@ -221,5 +221,5 @@
         <parent link="hand_link"/>
         <child link="tendon_right_link"/>
-        <origin xyz="0 -1 5" rpy="-1.57 0 0"/>
+        <origin xyz="0 -0.01 0.05" rpy="-1.57 0 0"/>
         <axis xyz="1 0 0"/>
         <limit lower="0" upper="1.57" effort="1000" velocity="0.5"/>
@@ -228,36 +228,36 @@
     <link name="tendon_left_link">
         <visual>
-            <origin xyz="0 0 5" rpy="0 0 0"/>
-            <geometry>
-                <cylinder radius="0.25" length="3.8" />
+            <origin xyz="0 0 0.05" rpy="0 0 0"/>
+            <geometry>
+                <cylinder radius="0.0025" length="0.038" />
             </geometry>
             <material name="orange" />
         </visual>
         <collision>
-            <origin xyz="0 0 5" rpy="0 0 0"/>
-            <geometry>
-                <cylinder radius="0.25" length="3.8" />
-            </geometry>
-        </collision>
-        <xacro:inertial_cylinder mass="1" length="3.8" radius="0.25">
-            <origin xyz="0 0 5" rpy="0 0 0"/>
+            <origin xyz="0 0 0.05" rpy="0 0 0"/>
+            <geometry>
+                <cylinder radius="0.0025" length="0.038" />
+            </geometry>
+        </collision>
+        <xacro:inertial_cylinder mass="1" length="0.038" radius="0.0025">
+            <origin xyz="0 0 0.05" rpy="0 0 0"/>
         </xacro:inertial_cylinder>
     </link>
     <link name="tendon_right_link">
         <visual>
-            <origin xyz="0 0 5" rpy="0 0 0"/>
-            <geometry>
-                <cylinder radius="0.25" length="3.8" />
+            <origin xyz="0 0 0.05" rpy="0 0 0"/>
+            <geometry>
+                <cylinder radius="0.0025" length="0.038" />
             </geometry>
             <material name="orange" />
         </visual>
         <collision>
-            <origin xyz="0 0 5" rpy="0 0 0"/>
-            <geometry>
-                <cylinder radius="0.25" length="3.8" />
-            </geometry>
-        </collision>
-        <xacro:inertial_cylinder mass="1" length="3.8" radius="0.25">
-            <origin xyz="0 0 5" rpy="0 0 0"/>
+            <origin xyz="0 0 0.05" rpy="0 0 0"/>
+            <geometry>
+                <cylinder radius="0.0025" length="0.038" />
+            </geometry>
+        </collision>
+        <xacro:inertial_cylinder mass="1" length="0.038" radius="0.0025">
+            <origin xyz="0 0 0.05" rpy="0 0 0"/>
         </xacro:inertial_cylinder>
     </link>
@@ -266,5 +266,5 @@
         <parent link="grip_left_link"/>
         <child link="finger_left_link"/>
-        <origin xyz="0 0 5.5" rpy="1.57 0 0"/>
+        <origin xyz="0 0 0.055" rpy="1.57 0 0"/>
         <axis xyz="-1 0 0"/>
         <limit lower="-1.57" upper="0" effort="1000" velocity="0.5"/>
@@ -274,5 +274,5 @@
         <parent link="grip_right_link"/>
         <child link="finger_right_link"/>
-        <origin xyz="0 0 5.5" rpy="-1.57 0 0"/>
+        <origin xyz="0 0 0.055" rpy="-1.57 0 0"/>
         <axis xyz="-1 0 0"/>
         <limit lower="0" upper="1.57" effort="1000" velocity="0.5"/>
@@ -281,36 +281,36 @@
     <link name="finger_left_link">
         <visual>
-            <origin xyz="0 -0.5 3" rpy="0 0 0"/>
-            <geometry>
-                <box size="0.5 2 6.2" />
+            <origin xyz="0 -0.005 0.03" rpy="0 0 0"/>
+            <geometry>
+                <box size="0.005 0.02 0.062" />
             </geometry>
             <material name="red" />
         </visual>
         <collision>
-            <origin xyz="0 -0.5 3" rpy="0 0 0"/>
-            <geometry>
-                <box size="0.5 2 6.2" />
-            </geometry>
-        </collision>
-        <xacro:inertial_box mass="1" x="0.5" y="2" z="6.2">
-            <origin xyz="0 -0.5 3" rpy="0 0 0"/>
+            <origin xyz="0 -0.005 0.03" rpy="0 0 0"/>
+            <geometry>
+                <box size="0.005 0.02 0.062" />
+            </geometry>
+        </collision>
+        <xacro:inertial_box mass="1" x="0.005" y="0.02" z="0.062">
+            <origin xyz="0 -0.005 0.03" rpy="0 0 0"/>
         </xacro:inertial_box>
     </link>
     <link name="finger_right_link">
         <visual>
-            <origin xyz="0 0.5 3" rpy="0 0 0"/>
-            <geometry>
-                <box size="0.5 -2 6.2" />
+            <origin xyz="0 0.005 0.03" rpy="0 0 0"/>
+            <geometry>
+                <box size="0.005 -0.02 0.062" />
             </geometry>
             <material name="red" />
         </visual>
         <collision>
-            <origin xyz="0 0.5 3" rpy="0 0 0"/>
-            <geometry>
-                <box size="0.5 -2 6.2" />
-            </geometry>
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
Commit message: Added stl files.. need to be rotated in the stl file... do later

File: src/learm_ros2_description/urdf/scaledLearm.urdf.xacro (robot description, xacro)
@@ -14,9 +14,6 @@
             <origin xyz="0 0 0.035" rpy="0 0 0"/>
             <geometry>
-                <box size="0.16 0.29 0.07" />
-            </geometry>
-            <material name="green">
-                <color rgba="0.2 1 0.2 1"/>
-            </material>
+                <mesh filename="package://learm_ros2_description/meshes/base.stl"/>
+            </geometry>
         </visual>
         <collision>
@@ -41,9 +38,6 @@
             <origin xyz="0 0 0" rpy="0 0 0"/>
             <geometry>
-                <box size="0.042 0.041 0.022" />
-            </geometry>
-            <material name="black">
-                <color rgba="0 0 0 0.91"/>
-            </material>
+                <mesh filename="package://learm_ros2_description/meshes/shoulder.stl"/>
+            </geometry>
         </visual>
         <collision>
@@ -68,7 +62,6 @@
             <origin xyz="0 0.015 0.07" rpy="0 0 0"/>
             <geometry>
-                <box size="0.055 0.03 0.13" />
-            </geometry>
-            <material name="blue" />
+                <mesh filename="package://learm_ros2_description/meshes/humerus.stl"/>
+            </geometry>
         </visual>
         <collision>
@@ -93,7 +86,6 @@
             <origin xyz="0 0 0.055" rpy="0 0 0"/>
             <geometry>
-                <box size="0.055 0.03 0.11" />
-            </geometry>
-            <material name="blue" />
+                <mesh filename="package://learm_ros2_description/meshes/forearm.stl"/>
+            </geometry>
         </visual>
         <collision>
@@ -118,7 +110,6 @@
             <origin xyz="0 0.015 0.0325" rpy="0 0 0"/>
             <geometry>
-                <box size="0.055 0.05 0.075" />
-            </geometry>
-            <material name="blue" />
+                <mesh filename="package://learm_ros2_description/meshes/wrist.stl"/>
+            </geometry>
         </visual>
         <collision>
@@ -143,7 +134,6 @@
             <origin xyz="0.015 -0.015 0.02" rpy="0 0 0"/>
             <geometry>
-                <box size="0.05 0.055 0.04" />
-            </geometry>
-            <material name="blue" />
+                <mesh filename="package://learm_ros2_description/meshes/hand.stl"/>
+            </geometry>
         </visual>
         <collision>
@@ -177,13 +167,12 @@
             <origin xyz="0 0 0.03" rpy="0 0 0"/>
             <geometry>
+                <mesh filename="package://learm_ros2_description/meshes/carpal-left.stl"/>
+            </geometry>
+        </visual>
+        <collision>
+            <origin xyz="0 0 0.03" rpy="0 0 0"/>
+            <geometry>
                 <box size="0.005 -0.028 0.05" />
             </geometry>
-            <material name="orange" />
-        </visual>
-        <collision>
-            <origin xyz="0 0 0.03" rpy="0 0 0"/>
-            <geometry>
-                <box size="0.005 -0.028 0.05" />
-            </geometry>
         </collision>
         <xacro:inertial_box mass="1" x="0.005" y="-0.028" z="0.05">
@@ -195,7 +184,6 @@
             <origin xyz="0 0 0.03" rpy="0 0 0"/>
             <geometry>
-                <box size="0.005 0.028 0.05" />
-            </geometry>
-            <material name="orange" />
+                <mesh filename="package://learm_ros2_description/meshes/carpal-right.stl"/>
+            </geometry>
         </visual>
         <collision>
@@ -230,7 +218,24 @@
             <origin xyz="0 0 0.05" rpy="0 0 0"/>
             <geometry>
+                <mesh filename="package://learm_ros2_description/meshes/tendon.stl"/>
+            </geometry>
+        </visual>
+        <collision>
+            <origin xyz="0 0 0.05" rpy="0 0 0"/>
+            <geometry>
                 <cylinder radius="0.0025" length="0.038" />
             </geometry>
-            <material name="orange" />
+            <material name="blue" />
+        </collision>
+        <xacro:inertial_cylinder mass="1" length="0.038" radius="0.0025">
+            <origin xyz="0 0 0.05" rpy="0 0 0"/>
+        </xacro:inertial_cylinder>
+    </link>
+    <link name="tendon_right_link">
+        <visual>
+            <origin xyz="0 0 0.05" rpy="0 0 0"/>
+            <geometry>
+                <mesh filename="package://learm_ros2_description/meshes/tendon.stl"/>
+            </geometry>
         </visual>
         <collision>
@@ -239,22 +244,5 @@
                 <cylinder radius="0.0025" length="0.038" />
             </geometry>
-        </collision>
-        <xacro:inertial_cylinder mass="1" length="0.038" radius="0.0025">
-            <origin xyz="0 0 0.05" rpy="0 0 0"/>
-        </xacro:inertial_cylinder>
-    </link>
-    <link name="tendon_right_link">
-        <visual>
-            <origin xyz="0 0 0.05" rpy="0 0 0"/>
-            <geometry>
-                <cylinder radius="0.0025" length="0.038" />
-            </geometry>
-            <material name="orange" />
-        </visual>
-        <collision>
-            <origin xyz="0 0 0.05" rpy="0 0 0"/>
-            <geometry>
-                <cylinder radius="0.0025" length="0.038" />
-            </geometry>
+            <material name="blue" />
         </collision>
         <xacro:inertial_cylinder mass="1" length="0.038" radius="0.0025">
@@ -283,7 +271,6 @@
             <origin xyz="0 -0.005 0.03" rpy="0 0 0"/>
             <geometry>
-                <box size="0.005 0.02 0.062" />
-            </geometry>
-            <material name="red" />
+                <mesh filename="package://learm_ros2_description/meshes/finger.stl"/>
+            </geometry>
         </visual>
         <collision>
@@ -301,7 +288,6 @@
             <origin xyz="0 0.005 0.03" rpy="0 0 0"/>
             <geometry>
-                <box size="0.005 -0.02 0.062" />
-            </geometry>
-            <material name="red" />
+                <mesh filename="package://learm_ros2_description/meshes/finger.stl"/>
+            </geometry>
         </visual>
         <collision>
