Commit message: Added collisions to URDF. Inertial boxes need to be raised by half of the z height

File: src/learm_ros2_description/urdf/example_include.xacro (robot description, xacro)
@@ -17,4 +17,7 @@
     <material name="red">
         <color rgba="1 0 0 1"/>
+    </material>
+    <material name="green">
+        <color rgba="0 1 0 1"/>
     </material>
     <!-- Specify some standard inertial calculations https://en.wikipedia.org/wiki/List_of_moments_of_inertia -->

File: src/learm_ros2_description/urdf/learm.urdf.xacro (robot description, xacro)
@@ -8,5 +8,14 @@
         <mesh filename="package://learm_ros2_description/meshes/base.stl"/>
       </geometry>
-    </visual>
+      <material name="black"/>
+    </visual>
+    <collision>
+      <geometry>
+        <mesh filename="package://learm_ros2_description/meshes/base.stl"/>
+      </geometry>
+    </collision>
+    <xacro:inertial_box mass="500" x="0.28291523" y="0.16" z="0.0795">
+      <origin xyz="0 0 0" rpy="0 0 0"/>
+    </xacro:inertial_box>
   </link>
   <joint name="shoulder_pan" type="revolute">
@@ -22,5 +31,14 @@
         <mesh filename="package://learm_ros2_description/meshes/shoulder.stl"/>
       </geometry>
-    </visual>
+      <material name="green"/>
+    </visual>
+    <collision>
+      <geometry>
+        <mesh filename="package://learm_ros2_description/meshes/shoulder.stl"/>
+      </geometry>
+    </collision>
+    <xacro:inertial_box mass="50" x="0.08100046" y="0.081" z="0.03901956">
+      <origin xyz="0 0 0" rpy="0 0 0"/>
+    </xacro:inertial_box>
   </link>
   <joint name="shoulder_lift" type="revolute">
@@ -36,5 +54,14 @@
         <mesh filename="package://learm_ros2_description/meshes/humerus.stl"/>
       </geometry>
-    </visual>
+      <material name="blue"/>
+    </visual>
+    <collision>
+      <geometry>
+        <mesh filename="package://learm_ros2_description/meshes/humerus.stl"/>
+      </geometry>
+    </collision>
+    <xacro:inertial_box mass="200" x="0.025" y="0.056" z="0.12900001">
+      <origin xyz="0 0 0" rpy="0 0 0"/>
+    </xacro:inertial_box>
   </link>
   <joint name="elbow" type="revolute">
@@ -50,5 +77,14 @@
         <mesh filename="package://learm_ros2_description/meshes/forearm.stl"/>
       </geometry>
-    </visual>
+      <material name="blue"/>
+    </visual>
+    <collision>
+      <geometry>
+        <mesh filename="package://learm_ros2_description/meshes/forearm.stl"/>
+      </geometry>
+    </collision>
+    <xacro:inertial_box mass="200" x="0.025" y="0.056" z="0.11098956">
+      <origin xyz="0 0 0" rpy="0 0 0"/>
+    </xacro:inertial_box>
   </link>
   <joint name="wrist_flex" type="revolute">
@@ -64,5 +100,14 @@
         <mesh filename="package://learm_ros2_description/meshes/wrist.stl"/>
       </geometry>
-    </visual>
+      <material name="blue"/>
+    </visual>
+    <collision>
+      <geometry>
+        <mesh filename="package://learm_ros2_description/meshes/wrist.stl"/>
+      </geometry>
+    </collision>
+    <xacro:inertial_box mass="200" x="0.0583" y="0.0456" z="0.0711">
+      <origin xyz="0 0 0" rpy="0 0 0"/>
+    </xacro:inertial_box>
   </link>
   <joint name="wrist_roll" type="revolute">
@@ -78,5 +123,14 @@
         <mesh filename="package://learm_ros2_description/meshes/hand.stl"/>
       </geometry>
-    </visual>
+      <material name="black"/>
+    </visual>
+    <collision>
+      <geometry>
+        <mesh filename="package://learm_ros2_description/meshes/hand.stl"/>
+      </geometry>
+    </collision>
+    <xacro:inertial_box mass="200" x="0.05439999" y="0.05563842" z="0.056">
+      <origin xyz="0 0 0" rpy="0 0 0"/>
+    </xacro:inertial_box>
   </link>
   <!-- Gripper specific links: -->
@@ -86,5 +140,14 @@
         <mesh filename="package://learm_ros2_description/meshes/carpal-left.stl"/>
       </geometry>
-    </visual>
+      <material name="orange"/>
+    </visual>
+    <collision>
+      <geometry>
+        <mesh filename="package://learm_ros2_description/meshes/carpal-left.stl"/>
+      </geometry>
+    </collision>
+    <xacro:inertial_box mass="10" x="0.003" y="0.02781075" z="0.04949519">
+      <origin xyz="0 0 0" rpy="0 0 0"/>
+    </xacro:inertial_box>
   </link>
   <link name="grip_right_link">
@@ -93,5 +156,14 @@
         <mesh filename="package://learm_ros2_description/meshes/carpal-right.stl"/>
       </geometry>
-    </visual>
+      <material name="orange"/>
+    </visual>
+    <collision>
+      <geometry>
+        <mesh filename="package://learm_ros2_description/meshes/carpal-right.stl"/>
+      </geometry>
+    </collision>
+    <xacro:inertial_box mass="10" x="0.00824992" y="0.02793942" z="0.04944835">
+      <origin xyz="0 0 0" rpy="0 0 0"/>
+    </xacro:inertial_box>
   </link>
   <link name="tendon_left_link">
@@ -100,5 +172,14 @@
         <mesh filename="package://learm_ros2_description/meshes/tendon.stl"/>
       </geometry>
-    </visual>
+      <material name="orange"/>
+    </visual>
+    <collision>
+      <geometry>
+        <mesh filename="package://learm_ros2_description/meshes/tendon.stl"/>
+      </geometry>
+    </collision>
+    <xacro:inertial_box mass="5" x="0.012" y="0.00710179" z="0.03599977">
+      <origin xyz="0 0 0" rpy="0 0 0"/>
+    </xacro:inertial_box>
   </link>
   <link name="tendon_right_link">
@@ -107,5 +188,14 @@
         <mesh filename="package://learm_ros2_description/meshes/tendon.stl"/>
       </geometry>
-    </visual>
+      <material name="orange"/>
+    </visual>
+    <collision>
+      <geometry>
+        <mesh filename="package://learm_ros2_description/meshes/tendon.stl"/>
+      </geometry>
+    </collision>
+    <xacro:inertial_box mass="5" x="0.012" y="0.00710179" z="0.03599977">
+      <origin xyz="0 0 0" rpy="0 0 0"/>
+    </xacro:inertial_box>
   </link>
   <link name="finger_left_link">
@@ -114,13 +204,32 @@
         <mesh filename="package://learm_ros2_description/meshes/finger.stl"/>
       </geometry>
-    </visual>
+      <material name="red"/>
+    </visual>
+    <collision>
+      <geometry>
+        <mesh filename="package://learm_ros2_description/meshes/finger.stl"/>
+      </geometry>
+    </collision>
+    <xacro:inertial_box mass="10" x="0.006" y="0.02043952" z="0.05933856">
+      <origin xyz="0 0 0" rpy="0 0 0"/>
+    </xacro:inertial_box>
   </link>
   <link name="finger_right_link">
     <visual>
-      <origin rpy="0 0 3.14159"/>
-      <geometry>
-        <mesh filename="package://learm_ros2_description/meshes/finger.stl"/>
-      </geometry>
-    </visual>
+      <origin rpy="0 0 ${pi}"/>
+      <geometry>
+        <mesh filename="package://learm_ros2_description/meshes/finger.stl"/>
+      </geometry>
+      <material name="red"/>
+    </visual>
+    <collision>
+      <origin rpy="0 0 ${pi}"/>
+      <geometry>
+        <mesh filename="package://learm_ros2_description/meshes/finger.stl"/>
+      </geometry>
+    </collision>
+    <xacro:inertial_box mass="10" x="0.006" y="0.02043952" z="0.05933856">
+      <origin xyz="0 0 ${pi}" rpy="0 0 0"/>
+    </xacro:inertial_box>
   </link>
   <!-- Gripper specific joints: -->

File: src/learm_ros2_description/urdf/scaledLearm.urdf.xacro (robot description, xacro)
@@ -12,13 +12,14 @@
     <link name="base_link">
         <visual>
-            <origin xyz="0 0 0.035" rpy="0 0 0"/>
+            <origin xyz="0 0.07 0" rpy="0 0 ${pi/2}"/>
             <geometry>
                 <mesh filename="package://learm_ros2_description/meshes/base.stl"/>
             </geometry>
-        </visual>
-        <collision>
-            <origin xyz="0 0 0.035" rpy="0 0 0"/>
-            <geometry>
-                <box size="0.16 0.29 0.07" />
+            <material name="black" />
+        </visual>
+        <collision>
+            <origin xyz="0 0.07 0" rpy="0 0 ${pi/2}"/>
+            <geometry>
+                <mesh filename="package://learm_ros2_description/meshes/base.stl"/>
             </geometry>
         </collision>
@@ -36,13 +37,14 @@
     <link name="shoulder_link">
         <visual>
-            <origin xyz="0 0 0" rpy="0 0 0"/>
+            <origin xyz="0 0 0" rpy="0 0 ${-pi/2}"/>
             <geometry>
                 <mesh filename="package://learm_ros2_description/meshes/shoulder.stl"/>
             </geometry>
-        </visual>
-        <collision>
-            <origin xyz="0 0 0" rpy="0 0 0"/>
-            <geometry>
-                <box size="0.042 0.041 0.022" />
+            <material name="green" />
+        </visual>
+        <collision>
+            <origin xyz="0 0 0" rpy="0 0 ${-pi/2}"/>
+            <geometry>
+                <mesh filename="package://learm_ros2_description/meshes/shoulder.stl"/>
             </geometry>
         </collision>
@@ -60,13 +62,14 @@
     <link name="humerus_link">
         <visual>
-            <origin xyz="0 0.015 0.07" rpy="0 0 0"/>
+            <origin xyz="0 0.015 0.07" rpy="0 0 ${pi/2}"/>
             <geometry>
                 <mesh filename="package://learm_ros2_description/meshes/humerus.stl"/>
             </geometry>
-        </visual>
-        <collision>
-            <origin xyz="0 0.015 0.07" rpy="0 0 0"/>
-            <geometry>
-                <box size="0.055 0.03 0.13" />
+            <material name="blue" />
+        </visual>
+        <collision>
+            <origin xyz="0 0.015 0.07" rpy="0 0 ${pi/2}"/>
+            <geometry>
+                <mesh filename="package://learm_ros2_description/meshes/humerus.stl"/>
             </geometry>
         </collision>
@@ -84,13 +87,14 @@
     <link name="forearm_link">
         <visual>
-            <origin xyz="0 0 0.055" rpy="0 0 0"/>
+            <origin xyz="0 0 0.055" rpy="0 0 ${pi/2}"/>
             <geometry>
                 <mesh filename="package://learm_ros2_description/meshes/forearm.stl"/>
             </geometry>
-        </visual>
-        <collision>
-            <origin xyz="0 0 0.055" rpy="0 0 0"/>
-            <geometry>
-                <box size="0.055 0.03 0.11" />
+            <material name="blue" />
+        </visual>
+        <collision>
+            <origin xyz="0 0 0.055" rpy="0 0 ${pi/2}"/>
+            <geometry>
+                <mesh filename="package://learm_ros2_description/meshes/forearm.stl"/>
             </geometry>
         </collision>
@@ -112,4 +116,5 @@
                 <mesh filename="package://learm_ros2_description/meshes/wrist.stl"/>
             </geometry>
+            <material name="blue" />
         </visual>
         <collision>
@@ -136,4 +141,5 @@
                 <mesh filename="package://learm_ros2_description/meshes/hand.stl"/>
             </geometry>
+            <material name="black" />
         </visual>
         <collision>
@@ -169,4 +175,5 @@
                 <mesh filename="package://learm_ros2_description/meshes/carpal-left.stl"/>
             </geometry>
+            <material name="orange" />
         </visual>
         <collision>
@@ -186,4 +193,5 @@
                 <mesh filename="package://learm_ros2_description/meshes/carpal-right.stl"/>
             </geometry>
+            <material name="orange" />
         </visual>
         <collision>
@@ -220,4 +228,5 @@
                 <mesh filename="package://learm_ros2_description/meshes/tendon.stl"/>
             </geometry>
+            <material name="orange" />
         </visual>
         <collision>
@@ -273,4 +282,5 @@
                 <mesh filename="package://learm_ros2_description/meshes/finger.stl"/>
             </geometry>
+            <material name="red" />
         </visual>
         <collision>
@@ -290,4 +300,5 @@
                 <mesh filename="package://learm_ros2_description/meshes/finger.stl"/>
             </geometry>
+            <material name="red" />
         </visual>
         <collision>
