Commit message: Added modeling for the hand

File: src/learm_ros2_description/urdf/learm.urdf.xacro (robot description, xacro)
@@ -1,8 +1,6 @@
-<?xml version="1.0" ?>
-<!-- =================================================================================== -->
-<!-- |    This document was autogenerated by xacro from src/learm_ros2_description/urdf/learm.urdf | -->
-<!-- |    EDITING THIS FILE BY HAND IS NOT RECOMMENDED                                 | -->
-<!-- =================================================================================== -->
-<robot name="learm">
+<?xml version="1.0"?>
+<robot xmlns:xacro="http://www.ros.org/wiki/xacro" name="learm">
+  <!-- Include some basic inertial shapes for reuse. -->
+  <xacro:include filename="example_include.xacro" />
   <link name="base_link">
     <visual>
@@ -12,4 +10,11 @@
     </visual>
   </link>
+  <joint name="shoulder_pan" type="revolute">
+    <parent link="base_link"/>
+    <child link="shoulder_link"/>
+    <origin xyz="0 0 0.059"/>
+    <axis xyz="0 0 1"/>
+    <limit lower="-1.57" upper="1.57" effort="1000" velocity="0.5"/>
+  </joint>
   <link name="shoulder_link">
     <visual>
@@ -19,4 +24,11 @@
     </visual>
   </link>
+  <joint name="shoulder_lift" type="revolute">
+    <parent link="shoulder_link"/>
+    <child link="humerus_link"/>
+    <origin xyz="-0.010 0 0.028"/>
+    <axis xyz="0 1 0"/>
+    <limit lower="-1.57" upper="1.57" effort="1000" velocity="0.5"/>
+  </joint>
   <link name="humerus_link">
     <visual>
@@ -26,4 +38,11 @@
     </visual>
   </link>
+  <joint name="elbow" type="revolute">
+    <parent link="humerus_link"/>
+    <child link="forearm_link"/>
+    <origin xyz="0 0 0.105"/>
+    <axis xyz="0 -1 0"/>
+    <limit lower="-1.57" upper="1.57" effort="1000" velocity="0.5"/>
+  </joint>
   <link name="forearm_link">
     <visual>
@@ -33,4 +52,11 @@
     </visual>
   </link>
+  <joint name="wrist_flex" type="revolute">
+    <parent link="forearm_link"/>
+    <child link="wrist_link"/>
+    <origin xyz="0 0 0.090"/>
+    <axis xyz="0 -1 0"/>
+    <limit lower="-1.57" upper="1.57" effort="1000" velocity="0.5"/>
+  </joint>
   <link name="wrist_link">
     <visual>
@@ -40,4 +66,11 @@
     </visual>
   </link>
+  <joint name="wrist_roll" type="revolute">
+    <parent link="wrist_link"/>
+    <child link="hand_link"/>
+    <origin xyz="0 0 0.060"/>
+    <axis xyz="0 0 1"/>
+    <limit lower="-1.57" upper="1.57" effort="1000" velocity="0.5"/>
+  </joint>
   <link name="hand_link">
     <visual>
@@ -47,4 +80,5 @@
     </visual>
   </link>
+  <!-- Gripper specific links: -->
   <link name="grip_left_link">
     <visual>
@@ -90,52 +124,18 @@
     </visual>
   </link>
-  <joint name="shoulder_pan" type="revolute">
-    <parent link="base_link"/>
-    <child link="shoulder_link"/>
-    <origin xyz="0 0 0.059"/>
-    <axis xyz="0 0 1"/>
-    <limit effort="1000" lower="-1.57" upper="1.57" velocity="0.5"/>
-  </joint>
-  <joint name="shoulder_lift" type="revolute">
-    <parent link="shoulder_link"/>
-    <child link="humerus_link"/>
-    <origin xyz="-0.010 0 0.028"/>
-    <axis xyz="0 1 0"/>
-    <limit effort="1000" lower="-1.57" upper="1.57" velocity="0.5"/>
-  </joint>
-  <joint name="elbow" type="revolute">
-    <parent link="humerus_link"/>
-    <child link="forearm_link"/>
-    <origin xyz="0 0 0.105"/>
-    <axis xyz="0 -1 0"/>
-    <limit effort="1000" lower="-1.57" upper="1.57" velocity="0.5"/>
-  </joint>
-  <joint name="wrist_flex" type="revolute">
-    <parent link="forearm_link"/>
-    <child link="wrist_link"/>
-    <origin xyz="0 0 0.090"/>
-    <axis xyz="0 -1 0"/>
-    <limit effort="1000" lower="-1.57" upper="1.57" velocity="0.5"/>
-  </joint>
-  <joint name="wrist_roll" type="revolute">
-    <parent link="wrist_link"/>
-    <child link="hand_link"/>
-    <origin xyz="0 0 0.060"/>
-    <axis xyz="0 0 1"/>
-    <limit effort="1000" lower="-1.57" upper="1.57" velocity="0.5"/>
-  </joint>
+  <!-- Gripper specific joints: -->
   <joint name="grip_left" type="revolute">
     <parent link="hand_link"/>
     <child link="grip_left_link"/>
-    <origin rpy="-1.57 0 0" xyz="0 +0.015 0.030"/>
+    <origin xyz="0 +0.015 0.030" rpy="-1.57 0 0"/>
     <axis xyz="-1 0 0"/>
-    <limit effort="1000" lower="-1.57" upper="0" velocity="0.5"/>
+    <limit lower="-1.57" upper="0" effort="1000" velocity="0.5"/>
   </joint>
   <joint name="grip_right" type="revolute">
     <parent link="hand_link"/>
     <child link="grip_right_link"/>
-    <origin rpy="1.57 0 0" xyz="0 -0.015 0.030"/>
+    <origin xyz="0 -0.015 0.030" rpy="1.57 0 0"/>
     <axis xyz="-1 0 0"/>
-    <limit effort="1000" lower="0" upper="1.57" velocity="0.5"/>
+    <limit lower="0" upper="1.57" effort="1000" velocity="0.5"/>
     <mimic joint="grip_left" multiplier="-1"/>
   </joint>
@@ -143,7 +143,7 @@
     <parent link="hand_link"/>
     <child link="tendon_left_link"/>
-    <origin rpy="-1.57 0 0" xyz="0 +0.005 0.050"/>
+    <origin xyz="0 +0.005 0.050" rpy="-1.57 0 0"/>
     <axis xyz="-1 0 0"/>
-    <limit effort="1000" lower="-1.57" upper="0" velocity="0.5"/>
+    <limit lower="-1.57" upper="0" effort="1000" velocity="0.5"/>
     <mimic joint="grip_left"/>
   </joint>
@@ -151,7 +151,7 @@
     <parent link="hand_link"/>
     <child link="tendon_right_link"/>
-    <origin rpy="1.57 0 0" xyz="0 -0.005 0.050"/>
+    <origin xyz="0 -0.005 0.050" rpy="1.57 0 0"/>
     <axis xyz="-1 0 0"/>
-    <limit effort="1000" lower="0" upper="1.57" velocity="0.5"/>
+    <limit lower="0" upper="1.57" effort="1000" velocity="0.5"/>
     <mimic joint="grip_left" multiplier="-1"/>
   </joint>
@@ -159,7 +159,7 @@
     <parent link="grip_left_link"/>
     <child link="finger_left_link"/>
-    <origin rpy="1.57 0 0" xyz="0 0 0.030"/>
+    <origin xyz="0 0 0.030" rpy="1.57 0 0"/>
     <axis xyz="-1 0 0"/>
-    <limit effort="1000" lower="-1.57" upper="0" velocity="0.5"/>
+    <limit lower="-1.57" upper="0" effort="1000" velocity="0.5"/>
     <mimic joint="grip_left" multiplier="-1"/>
   </joint>
@@ -167,7 +167,7 @@
     <parent link="grip_right_link"/>
     <child link="finger_right_link"/>
-    <origin rpy="-1.57 0 0" xyz="0 0 0.030"/>
+    <origin xyz="0 0 0.030" rpy="-1.57 0 0"/>
     <axis xyz="-1 0 0"/>
-    <limit effort="1000" lower="0" upper="1.57" velocity="0.5"/>
+    <limit lower="0" upper="1.57" effort="1000" velocity="0.5"/>
     <mimic joint="grip_left"/>
   </joint>

Commit message: inertial boxes adjusted to ~mostly~ proper spots

File: src/learm_ros2_description/urdf/learm.urdf.xacro (robot description, xacro)
@@ -16,5 +16,5 @@
     </collision>
     <xacro:inertial_box mass="500" x="0.28291523" y="0.16" z="0.0795">
-      <origin xyz="0 0 0" rpy="0 0 0"/>
+      <origin xyz="0 0 ${0.0795/2}" rpy="0 0 0"/>
     </xacro:inertial_box>
   </link>
@@ -39,5 +39,5 @@
     </collision>
     <xacro:inertial_box mass="50" x="0.08100046" y="0.081" z="0.03901956">
-      <origin xyz="0 0 0" rpy="0 0 0"/>
+      <origin xyz="0 0 ${0.03901956/2}" rpy="0 0 0"/>
     </xacro:inertial_box>
   </link>
@@ -62,5 +62,5 @@
     </collision>
     <xacro:inertial_box mass="200" x="0.025" y="0.056" z="0.12900001">
-      <origin xyz="0 0 0" rpy="0 0 0"/>
+      <origin xyz="0 0 ${0.12900001/2}" rpy="0 0 0"/>
     </xacro:inertial_box>
   </link>
@@ -85,5 +85,5 @@
     </collision>
     <xacro:inertial_box mass="200" x="0.025" y="0.056" z="0.11098956">
-      <origin xyz="0 0 0" rpy="0 0 0"/>
+      <origin xyz="0 0 ${0.11098956/2}" rpy="0 0 0"/>
     </xacro:inertial_box>
   </link>
@@ -108,5 +108,5 @@
     </collision>
     <xacro:inertial_box mass="200" x="0.0583" y="0.0456" z="0.0711">
-      <origin xyz="0 0 0" rpy="0 0 0"/>
+      <origin xyz="0 0 ${0.0711/2}" rpy="0 0 0"/>
     </xacro:inertial_box>
   </link>
@@ -131,5 +131,5 @@
     </collision>
     <xacro:inertial_box mass="200" x="0.05439999" y="0.05563842" z="0.056">
-      <origin xyz="0 0 0" rpy="0 0 0"/>
+      <origin xyz="0 0 ${0.056/2}" rpy="0 0 0"/>
     </xacro:inertial_box>
   </link>
@@ -148,5 +148,5 @@
     </collision>
     <xacro:inertial_box mass="10" x="0.003" y="0.02781075" z="0.04949519">
-      <origin xyz="0 0 0" rpy="0 0 0"/>
+      <origin xyz="0 0 ${0.04949519/2}" rpy="0 0 0"/>
     </xacro:inertial_box>
   </link>
@@ -164,5 +164,5 @@
     </collision>
     <xacro:inertial_box mass="10" x="0.00824992" y="0.02793942" z="0.04944835">
-      <origin xyz="0 0 0" rpy="0 0 0"/>
+      <origin xyz="0 0 ${0.04944835/2}" rpy="0 0 0"/>
     </xacro:inertial_box>
   </link>
@@ -180,5 +180,5 @@
     </collision>
     <xacro:inertial_box mass="5" x="0.012" y="0.00710179" z="0.03599977">
-      <origin xyz="0 0 0" rpy="0 0 0"/>
+      <origin xyz="0 0 ${0.03599977/2}" rpy="0 0 0"/>
     </xacro:inertial_box>
   </link>
@@ -196,5 +196,5 @@
     </collision>
     <xacro:inertial_box mass="5" x="0.012" y="0.00710179" z="0.03599977">
-      <origin xyz="0 0 0" rpy="0 0 0"/>
+      <origin xyz="0 0 ${0.03599977/2}" rpy="0 0 0"/>
     </xacro:inertial_box>
   </link>
@@ -212,5 +212,5 @@
     </collision>
     <xacro:inertial_box mass="10" x="0.006" y="0.02043952" z="0.05933856">
-      <origin xyz="0 0 0" rpy="0 0 0"/>
+      <origin xyz="0 0 ${0.05933856/2}" rpy="0 0 0"/>
     </xacro:inertial_box>
   </link>
@@ -230,5 +230,5 @@
     </collision>
     <xacro:inertial_box mass="10" x="0.006" y="0.02043952" z="0.05933856">
-      <origin xyz="0 0 ${pi}" rpy="0 0 0"/>
+      <origin xyz="0 0 ${0.05933856/2}" rpy="0 0 0"/>
     </xacro:inertial_box>
   </link>

Commit message: Stripped files down to remove extraneous urdf iterations

File: src/learm_ros2_description/urdf/learm.urdf.xacro (robot description, xacro)
@@ -2,5 +2,5 @@
 <robot xmlns:xacro="http://www.ros.org/wiki/xacro" name="learm">
   <!-- Include some basic inertial shapes for reuse. -->
-  <xacro:include filename="example_include.xacro" />
+  <xacro:include filename="macros.xacro" />
   <link name="base_link">
     <visual>

File: src/learm_ros2_description/urdf/macros.xacro (robot description, xacro)
@@ -1,5 +1,6 @@
 <?xml version="1.0"?>
-<robot xmlns:xacro="http://www.ros.org/wiki/xacro">
-    <!-- colors -->
+<robot xmlns:xacro="http://www.ros.org/wiki/xacro" >
+    <!-- This file is not a robot in and of itself, it just contains some useful tags that could be included in any robot -->
+    <!-- Specify some colours -->
     <material name="white">
         <color rgba="1 1 1 1"/>
@@ -17,126 +18,35 @@
         <color rgba="1 0 0 1"/>
     </material>
-  <!-- Macro for defining a joint and link -->
-  <xacro:macro name="joint_link" params="name parent child joint_origin axis lower upper velocity effort link_dims mass link_origin color">
-    <joint name="${name}" type="revolute">
-      <origin xyz="${joint_origin}" rpy="0 0 0"/>
-      <parent link="${parent}"/>
-      <child link="${child}"/>
-      <axis xyz="${axis}"/>
-      <limit lower="${lower}" upper="${upper}" velocity="${velocity}" effort="${effort}"/>
-    </joint>
-    <link name="${child}">
-      <xacro:visual_collision_inertial_box link_dims="${link_dims}" mass="${mass}" link_origin="${link_origin}" color="${color}"/>
-    </link>
-  </xacro:macro>
-  <!-- Macro for defining a joint and link for the base -->
-  <xacro:macro name="base_joint_link">
-    <joint name="base_joint" type="fixed">
-      <origin xyz="1.5 1.0 0" rpy="0 0 0"/>
-      <parent link="world"/>
-      <child link="base_link"/>
-    </joint>
-    <link name="base_link">
-      <xacro:visual_collision_inertial_box link_dims="16 29 7" mass="500" link_origin="0 0 3.5" color="green"/>
-    </link>
-  </xacro:macro>
-  <!-- Macro for defining grip joint and link -->
-  <xacro:macro name="grip_joint_link" params="side">
-    <joint name="grip_${side}" type="revolute">
-      <origin xyz="${side == 'left' ? '-1.5' : '1.5'} 0 3" rpy="0 ${side == 'left' ? '-1.57' : '1.57'} 0"/>
-      <parent link="hand_link"/>
-      <child link="grip_${side}_link"/>
-      <axis xyz="0 -1 0"/>
-      <limit lower="${side == 'left' ? '-1.57' : '0'}" upper="${side == 'left' ? '0' : '1.57'}" effort="1000" velocity="0.5"/>
-      <xacro:mimic joint="grip_${side == 'left' ? 'right' : 'left'}" multiplier="${side == 'left' ? '-1' : '1'}"/>
-    </joint>
-    <link name="grip_${side}_link">
-      <xacro:visual_collision_inertial_box link_dims="${side == 'left' ? '2.8 0.5 5' : '-2.8 0.5 5'}" mass="1" link_origin="0 0 3" color="orange"/>
-    </link>
-  </xacro:macro>
-  <!-- Macro for defining tendon joint and link -->
-  <xacro:macro name="tendon_joint_link" params="side">
-    <joint name="tendon_${side}" type="revolute">
-      <origin xyz="${side == 'left' ? '-0.5' : '0.5'} 0 5" rpy="0 ${side == 'left' ? '-1.57' : '1.57'} 0"/>
-      <parent link="hand_link"/>
-      <child link="tendon_${side}_link"/>
-      <axis xyz="0 -1 0"/>
-      <limit lower="${side == 'left' ? '-1.57' : '0'}" upper="${side == 'left' ? '0' : '1.57'}" effort="1000" velocity="0.5"/>
-      <xacro:mimic joint="grip_left" multiplier="${side == 'left' ? '1' : '-1'}"/>
-    </joint>
-    <link name="tendon_${side}_link">
-      <xacro:visual_collision_inertial_cylinder radius="0.25" length="3.8" mass="1" link_origin="0 0 5" color="orange"/>
-    </link>
-  </xacro:macro>
-  <!-- Macro for defining finger joint and link -->
-  <xacro:macro name="finger_joint_link" params="side">
-    <joint name="finger_${side}" type="revolute">
-      <origin xyz="0 0 5.5" rpy="0 ${side == 'left' ? '1.57' : '-1.57'} 0"/>
-      <parent link="grip_${side}_link"/>
-      <child link="finger_${side}_link"/>
-      <axis xyz="0 -1 0"/>
-      <limit lower="${side == 'left' ? '-1.57' : '0'}" upper="${side == 'left' ? '0' : '1.57'}" effort="1000" velocity="0.5"/>
-      <xacro:mimic joint="grip_left" multiplier="${side == 'left' ? '-1' : '1'}"/>
-    </joint>
-    <link name="finger_${side}_link">
-      <xacro:visual_collision_inertial_box link_dims="${side == 'left' ? '2 0.5 6.2' : '-2 0.5 6.2'}" mass="1" link_origin="${side == 'left' ? '0.5 0 3' : '-0.5 0 3'}" color="red"/>
-    </link>
-  </xacro:macro>
-  <!-- Macro for defining visual, collision, and inertial properties of a link -->
-  <xacro:macro name="visual_collision_inertial_box" params="link_dims mass link_origin color">
-    <visual>
-      <origin xyz="${link_origin}" rpy="0 0 0"/>
-      <geometry>
-        <box size="${link_dims}" />
-      </geometry>
-      <material name="${color}"/>
-    </visual>
-    <collision>
-      <origin xyz="${link_origin}" rpy="0 0 0"/>
-      <geometry>
-        <box size="${link_dims}" />
-      </geometry>
-    </collision>
-    <xacro:inertial_box mass="${mass}" x="${link_dims[0]}" y="${link_dims[1]}" z="${link_dims[2]}">
-        <origin xyz="link_origin" rpy="0 0 0"/>
-    </xacro:inertial_box>
-  </xacro:macro>
-  <xacro:macro name="inertial_box" params="mass x y z *origin">
-    <inertial>
-        <xacro:insert_block name="origin"/>
-        <mass value="${mass}" />
-        <inertia ixx="${(1/12) * mass * (y*y+z*z)}" ixy="0.0" ixz="0.0"
-                iyy="${(1/12) * mass * (x*x+z*z)}" iyz="0.0"
-                izz="${(1/12) * mass * (x*x+y*y)}" />
-    </inertial>
-  </xacro:macro>
-  <!-- Macro for defining visual, collision, and inertial properties of a cylinder -->
-  <xacro:macro name="visual_collision_inertial_cylinder" params="radius length mass link_origin color">
-    <visual>
-      <origin xyz="${link_origin}" rpy="0 0 0"/>
-      <geometry>
-        <cylinder radius="${radius}" length="${length}" />
-      </geometry>
-      <material name="${color}"/>
-    </visual>
-    <collision>
-      <origin xyz="${link_origin}" rpy="0 0 0"/>
-      <geometry>
-        <cylinder radius="${radius}" length="${length}" />
-      </geometry>
-    </collision>
-    <xacro:inertial_cylinder mass="${mass}" length="${length}" radius="${radius}">
-        <origin xyz="${link_origin}" rpy="0 0 0"/>
-    </xacro:inertial_cylinder>
-  </xacro:macro>
-  <!-- Macro for defining inertial properties of a cylinder -->
-  <xacro:macro name="inertial_cylinder" params="mass length radius *origin">
-    <inertial>
-        <xacro:insert_block name="origin"/>
-        <mass value="${mass}" />
-        <inertia ixx="${(1/12) * mass * (3*radius*radius + length*length)}" ixy="0.0" ixz="0.0"
-                iyy="${(1/12) * mass * (3*radius*radius + length*length)}" iyz="0.0"
-                izz="${(1/2) * mass * (radius*radius)}" />
-    </inertial>
-  </xacro:macro>
+    <material name="green">
+        <color rgba="0 1 0 1"/>
+    </material>
+    <!-- Specify some standard inertial calculations https://en.wikipedia.org/wiki/List_of_moments_of_inertia -->
+    <!-- These make use of xacro's mathematical functionality -->
+    <xacro:macro name="inertial_sphere" params="mass radius *origin">
+        <inertial>
+            <xacro:insert_block name="origin"/>
+            <mass value="${mass}" />
+            <inertia ixx="${(2/5) * mass * (radius*radius)}" ixy="0.0" ixz="0.0"
+                    iyy="${(2/5) * mass * (radius*radius)}" iyz="0.0"
+                    izz="${(2/5) * mass * (radius*radius)}" />
+        </inertial>
+    </xacro:macro>
+    <xacro:macro name="inertial_box" params="mass x y z *origin">
+        <inertial>
+            <xacro:insert_block name="origin"/>
+            <mass value="${mass}" />
+            <inertia ixx="${(1/12) * mass * (y*y+z*z)}" ixy="0.0" ixz="0.0"
+                    iyy="${(1/12) * mass * (x*x+z*z)}" iyz="0.0"
+                    izz="${(1/12) * mass * (x*x+y*y)}" />
+        </inertial>
+    </xacro:macro>
+    <xacro:macro name="inertial_cylinder" params="mass length radius *origin">
+        <inertial>
+            <xacro:insert_block name="origin"/>
+            <mass value="${mass}" />
+            <inertia ixx="${(1/12) * mass * (3*radius*radius + length*length)}" ixy="0.0" ixz="0.0"
+                    iyy="${(1/12) * mass * (3*radius*radius + length*length)}" iyz="0.0"
+                    izz="${(1/2) * mass * (radius*radius)}" />
+        </inertial>
+    </xacro:macro>
 </robot>
